File: design files/panel/hagiwo_double_seq.kicad_pcb (KiCad board)
At the start: 2 copper layers, 29.9 x 128.4 mm, 6 parts

Commit message: WIP
Parts:
- removed the G*** at (15.6, 65.3) (x6)
- added G*** (x2): LOGO, LOGO, F.Cu at (146.0, 92.3)
Other:
- board size 29.9 x 128.4 mm -> 30 x 128.4 mm
- net class Default removed
- rule pad_to_mask_clearance: 0.2 -> 0
